File: hardware/macropad.kicad_pcb (KiCad board)
At the start: 2 copper layers, 23 parts, among them J1 OLED_128x32, SW1 RotaryEncoder_Switch, U1 Raspberry_Pi_Pico

Commit message: wip
Parts:
- moved U1 18.3 mm to (39.5, 40.8)
- moved J1 6.01 mm to (72.4, 14.5)
- moved D10 0.61 mm to (128.0, 45.7)
- moved D2 0.61 mm to (89.9, 45.7)
- moved D3 0.61 mm to (108.9, 45.7)
- moved D4 0.61 mm to (70.8, 64.8)
- moved D5 0.61 mm to (89.9, 64.8)
- moved D6 0.61 mm to (108.9, 64.7)
- moved D7 0.61 mm to (70.8, 83.8)
- moved D8 0.61 mm to (89.9, 83.8)
- moved D9 0.61 mm to (108.9, 83.8)
- moved D1 0.55 mm to (70.9, 45.7)
Routing:
- net Net-(D9-A): track 3.81 -> 3.21 mm
- net Net-(D8-A): track 3.81 -> 3.21 mm
- net Net-(D7-A): track 3.81 -> 3.21 mm
- net Net-(D6-A): track 3.78 -> 3.17 mm
- net Net-(D5-A): track 3.81 -> 3.21 mm
- net Net-(D4-A): track 3.81 -> 3.21 mm
- net Net-(D3-A): track 3.81 -> 3.21 mm
- net Net-(D2-A): track 3.81 -> 3.21 mm
- net Net-(D10-A): track 3.81 -> 3.21 mm
Other:
- board outline added: 106.5 x 78.5 mm
